File: VerdiRT7_MainPCB.sch (EAGLE design)
At the start: 193 parts, among them J101 503480_1400, J102 BM04B-SRSS-TB(LF)(SN), J103 DF13-4P-1.25DSA, J104 1050270001, J105 503480_0400, J106 503480_0600, J201 DF58-2P-1.2V(21), J301 20021321-00010C4LF, J302 20021321-00010C4LF, J303 BM02B-SRSS-TB(LF)(SN), J401 52559-0652, Q201 SISA01DN-T1-GE3, Q301 SIZ322DT-T1-GE3, Q302 SIZ322DT-T1-GE3, Q303 SIZ322DT-T1-GE3, Q304 SIZ322DT-T1-GE3, Q305 SIZ322DT-T1-GE3, Q306 SIZ322DT-T1-GE3, SW101 SKRHABE010, SW102 SKQYACE010, SW201 AYZ0102AGRLC, U101 MCP1416T-E/OT, U102 MCP6001T-I/LT, U103 MCP6001T-I/LT, U104 R5F564MLDDFP#V1-ND, U105 MR20H40CDF, U201 TLV1117-50CDRJR, U202 TLV1117-33CDRJR, U301 74LVC2G08DC, U302 RT9625AZQW, U303 74LVC2G08DC, U304 RT9625AZQW, U305 74LVC2G08DC, U306 RT9625AZQW, U401 MCP1416T-E/OT, U402 MCP6001T-I/LT, U403 MCP1416T-E/OT, U404 MCP1416T-E/OT, U405 MCP6001T-I/LT, U501 ICM-20602, X101 NX3225SA-12.000M-STD-CSR-1

Commit message: updated: 捨て基板や認識マークを追加．発注データ作成
Parts:
- added S1, S2: BASE_HOLE, MountingSymbol:BASE_HOLE
- added S3: GUIDE_HOLE_1, MountingSymbol:GUIDE_HOLE_1
- added S4: GUIDE_HOLE_2, MountingSymbol:GUIDE_HOLE_2
- added S5: RECOG_MARK_1, MountingSymbol:RECOG_MARK_1
- added S6: RECOG_MARK_2, MountingSymbol:RECOG_MARK_2
- added S7: RECOG_MARK_3, MountingSymbol:RECOG_MARK_3
Changed lines of the file:
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@@
 <layer number="54" name="bGND_GNDA" color="1" fill="9" visible="no" active="no"/>
 <layer number="56" name="wert" color="7" fill="1" visible="no" active="no"/>
+<layer number="57" name="tCAD" color="7" fill="1" visible="no" active="no"/>
+<layer number="88" name="SimResults" color="9" fill="1" visible="yes" active="yes"/>
+<layer number="89" name="SimProbes" color="9" fill="1" visible="yes" active="yes"/>
 <layer number="90" name="Modules" color="5" fill="1" visible="yes" active="yes"/>
 <layer number="91" name="Nets" color="2" fill="1" visible="yes" active="yes"/>
@@
 <layer number="97" name="Info" color="7" fill="1" visible="yes" active="yes"/>
 <layer number="98" name="Guide" color="6" fill="1" visible="yes" active="yes"/>
+<layer number="99" name="SpiceOrder" color="7" fill="1" visible="no" active="no"/>
 <layer number="100" name="Muster" color="7" fill="1" visible="no" active="no"/>
 <layer number="101" name="Bemassung" color="7" fill="1" visible="yes" active="yes"/>
@@
 <layer number="106" name="bPlate" color="7" fill="1" visible="yes" active="yes"/>
 <layer number="107" name="Crop" color="7" fill="1" visible="yes" active="yes"/>
+<layer number="108" name="fp8" color="7" fill="1" visible="no" active="yes"/>
+<layer number="109" name="fp9" color="7" fill="1" visible="no" active="yes"/>
+<layer number="110" name="fp0" color="7" fill="1" visible="no" active="yes"/>
+<layer number="111" name="LPC17xx" color="7" fill="1" visible="no" active="yes"/>
+<layer number="112" name="tSilk" color="7" fill="1" visible="no" active="yes"/>
+<layer number="113" name="IDFDebug" color="7" fill="1" visible="no" active="yes"/>
 <layer number="116" name="Patch_BOT" color="9" fill="4" visible="yes" active="yes"/>
 <layer number="121" name="_tsilk" color="7" fill="1" visible="yes" active="yes"/>
 <layer number="122" name="_bsilk" color="7" fill="1" visible="yes" active="yes"/>
+<layer number="123" name="tTestmark" color="7" fill="1" visible="no" active="yes"/>
+<layer number="124" name="bTestmark" color="7" fill="1" visible="no" active="yes"/>
+<layer number="125" name="_tNames" color="7" fill="1" visible="no" active="yes"/>
+<layer number="126" name="_bNames" color="7" fill="1" visible="no" active="yes"/>
+<layer number="127" name="_tValues" color="7" fill="1" visible="no" active="yes"/>
+<layer number="128" name="_bValues" color="7" fill="1" visible="no" active="yes"/>
+<layer number="131" name="tAdjust" color="7" fill="1" visible="no" active="yes"/>
+<layer number="132" name="bAdjust" color="7" fill="1" visible="no" active="yes"/>
+<layer number="144" name="Drill_legend" color="7" fill="1" visible="no" active="yes"/>
+<layer number="150" name="Notes" color="7" fill="1" visible="no" active="yes"/>
 <layer number="151" name="HeatSink" color="7" fill="1" visible="yes" active="yes"/>
+<layer number="152" name="_bDocu" color="7" fill="1" visible="no" active="yes"/>
+<layer number="153" name="FabDoc1" color="7" fill="1" visible="no" active="yes"/>
+<layer number="154" name="FabDoc2" color="7" fill="1" visible="no" active="yes"/>
+<layer number="155" name="FabDoc3" color="7" fill="1" visible="no" active="yes"/>
+<layer number="199" name="Contour" color="7" fill="1" visible="no" active="yes"/>
 <layer number="200" name="200bmp" color="1" fill="10" visible="yes" active="yes"/>
 <layer number="201" name="201bmp" color="1" fill="10" visible="yes" active="yes"/>
@@
 <layer number="207" name="207bmp" color="8" fill="10" visible="yes" active="yes"/>
 <layer number="208" name="208bmp" color="9" fill="10" visible="yes" active="yes"/>
+<layer number="209" name="209bmp" color="7" fill="1" visible="no" active="yes"/>
+<layer number="210" name="210bmp" color="7" fill="1" visible="no" active="yes"/>
+<layer number="211" name="211bmp" color="7" fill="1" visible="no" active="yes"/>
+<layer number="212" name="212bmp" color="7" fill="1" visible="no" active="yes"/>
+<layer number="213" name="213bmp" color="7" fill="1" visible="no" active="yes"/>
+<layer number="214" name="214bmp" color="7" fill="1" visible="no" active="yes"/>
+<layer number="215" name="215bmp" color="7" fill="1" visible="no" active="yes"/>
+<layer number="216" name="216bmp" color="7" fill="1" visible="no" active="yes"/>
+<layer number="217" name="217bmp" color="18" fill="1" visible="no" active="no"/>
+<layer number="218" name="218bmp" color="19" fill="1" visible="no" active="no"/>
+<layer number="219" name="219bmp" color="20" fill="1" visible="no" active="no"/>
+<layer number="220" name="220bmp" color="21" fill="1" visible="no" active="no"/>
+<layer number="221" name="221bmp" color="22" fill="1" visible="no" active="no"/>
+<layer number="222" name="222bmp" color="23" fill="1" visible="no" active="no"/>
+<layer number="223" name="223bmp" color="24" fill="1" visible="no" active="no"/>
+<layer number="224" name="224bmp" color="25" fill="1" visible="no" active="no"/>
+<layer number="248" name="Housing" color="7" fill="1" visible="no" active="yes"/>
+<layer number="249" name="Edge" color="7" fill="1" visible="no" active="yes"/>
 <layer number="250" name="Descript" color="3" fill="1" visible="yes" active="yes"/>
 <layer number="251" name="SMDround" color="12" fill="11" visible="no" active="no"/>
@@
 <part name="U303" library="74xx-eu" deviceset="74LVC2G08" device="DC"/>
 <part name="U305" library="74xx-eu" deviceset="74LVC2G08" device="DC"/>
+<part name="S1" library="MountingSymbol" deviceset="BASE_HOLE" device=""/>
+<part name="S2" library="MountingSymbol" deviceset="BASE_HOLE" device=""/>
+<part name="S3" library="MountingSymbol" deviceset="GUIDE_HOLE" device="_1"/>
+<part name="S4" library="MountingSymbol" deviceset="GUIDE_HOLE" device="_2"/>
+<part name="S5" library="MountingSymbol" deviceset="RECOG_MARK" device="_1"/>
+<part name="S6" library="MountingSymbol" deviceset="RECOG_MARK" device="_2"/>
+<part name="S7" library="MountingSymbol" deviceset="RECOG_MARK" device="_3"/>
 </parts>
 <sheets>
@@
 </nets>
 </sheet>
+<sheet>
+<plain>
+<wire x1="0" y1="58.42" x2="0" y2="0" width="1.016" layer="98"/>
+<wire x1="0" y1="0" x2="78.74" y2="0" width="1.016" layer="98"/>
+<wire x1="78.74" y1="0" x2="78.74" y2="58.42" width="1.016" layer="98"/>
+<wire x1="78.74" y1="58.42" x2="0" y2="58.42" width="1.016" layer="98"/>
+<text x="5.08" y="2.54" size="6.4516" layer="98">designed by S.Hirai</text>
+</plain>
+<instances>
+<instance part="S1" gate="A" x="15.24" y="40.64"/>
+<instance part="S2" gate="A" x="31.75" y="40.64"/>
+<instance part="S3" gate="A" x="15.24" y="26.67"/>
+<instance part="S4" gate="A" x="31.75" y="26.67"/>
+<instance part="S5" gate="A" x="15.24" y="13.97"/>
+<instance part="S6" gate="A" x="36.83" y="13.97"/>
+<instance part="S7" gate="A" x="57.15" y="13.97"/>
+</instances>
+<busses>
+</busses>
+<nets>
+</nets>
+</sheet>
